File: cbus.sch (KiCad schematic (older format))
At the start: 32 parts, among them CON1 AVR-JTAG-10, J1 CBUS_IO, J2 Conn_02x20_Odd_Even, J3 Conn_02x05_Top_Bottom, J4 Conn_02x05_Top_Bottom, U1 SN74LVC8T245DWR, U2 SN74LVC8T245DWR, U3 SN74LVC8T245DWR, U4 SN74LVC8T245DWR, U5 MIC5365-1.2YC5-TR, U6 ICE40HX1K-VQ100, U7 MIC5504-3.3YM5-TR, U8 AT25SF041-SSHD-B

Commit message: Finish routing
Parts:
- removed U5: MIC5365-1.2YC5-TR, tinyfpga:SC-70-C5, symbol MIC5365-1.2YC5-TR
- removed U7: MIC5504-3.3YM5-TR, tinyfpga:SC-70-C5, symbol MIC5504-3.3YM5-TR
- added R? (x2): 1, Resistors_SMD:R_0805_HandSoldering, symbol R
- added U?: TPS76912, TO_SOT_Packages_SMD:SOT-23-5, symbol TPS76912
- added U?: TPS76933, TO_SOT_Packages_SMD:SOT-23-5, symbol TPS76933
- C2, C3: value 1uF -> 4.7uF
Connections:
- net +1V2: now also U?.5 (OUT)
- net +3V3: now also U?.1 (IN), U?.5 (OUT)
- net +5V: now also U?.1 (IN)
- net GND: now also U6.17 (GND), U6.23 (GND), U6.32 (GND), U6.39 (GND), U6.47 (GND), U6.5 (GND), U6.55 (GND), U6.70 (GND), U6.84 (GND), U6.98 (GND), R?.2, R?.2, U?.2 (GND), U?.2 (GND), U?.3 (~EN~), U?.3 (~EN~); no longer C2.2, C3.2
- new net: C2.2, R?.1
- new net: C3.2, R?.1
Other:
- moved on the sheet: C2, C3

Commit message: 1.0
Parts:
- U1, U2, U3, U4: footprint SN74LVC8T245DWR:SOIC127P1030X265-24N -> cbus:SOIC127P1030X265-24N
- gave numbers to parts that had none: 4

Commit message: Longboi
Parts:
- removed J3, J4: Conn_02x05_Top_Bottom, cbus:Pin_Header_Straight_2x05_Pitch2.54mm_Column_first, symbol Conn_02x05_Top_Bottom
- added J3, J4: DB9_Male, Connector_Dsub:DSUB-9_Male_Horizontal_P2.77x2.84mm_EdgePinOffset4.94mm_Housed_MountingHolesOffset7.48mm, symbol Connector:DB9_Male
- C1, C10, C11, C12, C13, C14, C15, C2, C3, C4, C5, C6, C7, C8, C9: symbol C -> cbus-rescue:C
- CON1: symbol AVR-JTAG-10 -> cbus-rescue:AVR-JTAG-10
- F1, F2: symbol Polyfuse -> cbus-rescue:Polyfuse
- J1: symbol CBUS_IO -> cbus_io:CBUS_IO
- J2: symbol Conn_02x20_Odd_Even -> cbus-rescue:Conn_02x20_Odd_Even
- R1, R2, R3, R4: symbol R -> cbus-rescue:R
- U1, U2, U3, U4: symbol SN74LVC8T245DWR -> SN74LVC8T245DWR:SN74LVC8T245DWR
- U5: symbol TPS76933 -> cbus-rescue:TPS76933
- U6: symbol ICE40HX1K-VQ100 -> ICE40HX1K-VQ100:ICE40HX1K-VQ100
- U7: symbol TPS76912 -> cbus-rescue:TPS76912
- U8: symbol AT25SF041-SSHD-B -> tinyfpga:AT25SF041-SSHD-B
Connections:
- net GND: now also J3.8, J4.8
- net P1B: now also J3.6
- net P1C: now also J3.9
- net P1D: now also J3.2
- net P1L: now also J3.3
- net P1R: now also J3.4
- net P1S: now also J3.7
- net P1U: now also J3.1
- net P2B: now also J4.6
- net P2C: now also J4.9
- net P2D: now also J4.2
- net P2L: now also J4.3
- net P2R: now also J4.4
- net P2S: now also J4.7
- net P2U: now also J4.1
- net at F1.1: now also J3.5
- net at F2.1: now also J4.5
Other:
- moved on the sheet: F1, F2
