File: cbus.kicad_pcb (KiCad board)
At the start: 2 copper layers, 180 x 149 mm, 39 parts, among them CON1 AVR-JTAG-10, J1 CBUS_IO, J2 Conn_02x20_Odd_Even, J3 DB9_Male, J4 DB9_Male, U1 SN74LVC8T245DWR, U2 SN74LVC8T245DWR, U3 SN74LVC8T245DWR, U4 SN74LVC8T245DWR, U5 TPS76933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

Commit message: Routing for v1.1
Parts:
- moved F2 114.6 mm to (183.8, 119.7), turned to 180 degrees
- moved F1 109.7 mm to (184.1, 70.0)
- moved J3 10.8 mm to (191.0, 81.0)
- moved J4 10.8 mm to (191.0, 131.0)
- moved svg2mod 10.8 mm to (194.0, 100.0)
- moved ? 8.32 mm to (195.0, 170.5)
- moved ? 6.50 mm to (195.0, 31.5)
- moved J1 0.71 mm to (34.5, 163.5)
- moved C12 0.36 mm to (63.1, 109.6)
Routing:
- net P2R: track 0.00 -> 171.6 mm, vias 0 -> 2
- net P2L: track 0.00 -> 163.2 mm, vias 0 -> 4
- net P2S: track 0.00 -> 161.5 mm, vias 0 -> 2
- net P1C: track 0.00 -> 160.4 mm
- net P2D: track 0.00 -> 159.9 mm, vias 0 -> 3
- net P2B: track 0.00 -> 155.0 mm, vias 0 -> 2
- net P2U: track 0.00 -> 153.8 mm, vias 0 -> 3
- net P1S: track 0.00 -> 152.7 mm
- net P1R: track 0.00 -> 151.2 mm, vias 0 -> 1
- net P1L: track 0.00 -> 148.5 mm, vias 0 -> 1
- net P1B: track 0.00 -> 147.6 mm
- net P1D: track 0.00 -> 147.3 mm, vias 0 -> 1
- net P1U: track 0.00 -> 144.1 mm
- net P2C: track 0.00 -> 139.0 mm, vias 0 -> 2
- net SDO: track 53.2 -> 102.7 mm, vias 2 -> 4
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Other:
- board size 180 x 149 mm -> 170 x 149 mm
- net class Default: via_drill 0.3 -> 0.4
